Commit message: feat: add scissor lift control, RViz config, Gazebo launch
- Added scissor_gazebo.launch.py with slider GUI and mapper
- Added scissor_lift_mapper.py: one-slider coupled joint control
- Added scissor_slider_gui.py: Tkinter GUI for scissor lift
- Updated URDF: scissor joints, IR frames, IMU, camera frames
- Fixed TF tree: world -> base_link static transform in all launches
- Fixed Gazebo bridge: correct joint_state topic path
- Updated RViz config: Fixed Frame = world

File: src/audix_pkg/urdf/audix.urdf (robot description, URDF)
Before this commit: robot audix, 24 links, 23 joints
Links:
- removed link RobotBody
- removed link ultrasonic_link
- added link camera_optical_link
- added link ir_back_link
- added link ir_front_left_link
- added link ir_front_link
- added link ir_front_right_link
- added link ir_left_link
- added link ir_right_link
- link back_left_wheel_link: mass 0.131907545752213 -> 0.131907512521704
- link back_right_wheel_link: mass 0.131907129758154 -> 0.131907120892093
- link base_link: mass 2.23789814285684 -> 2.23789814285683
- link bottom_stud_link: mass 0.00137057236420401 -> 0.00137057236420413
- link front_left_wheel_link: mass 0.131907084296385 -> 0.131907088712342
- link front_right_wheel_link: mass 0.131907400590731 -> 0.131907397861947
- link imu_link: mass 0.05 -> None; geometry 
- link left_link1: mass 0.0061541343895667 -> 0.00615413438956669
- link left_link3: mass 0.00615413438956668 -> 0.00615413438956673
- link left_link6: mass 0.00615413438956669 -> 0.00615413438956674
- link right_link2: mass 0.00615413438956677 -> 0.00615413438956663
- link right_link3: mass 0.00615413438956667 -> 0.00615413438956681
- link scissors_lift_base: mass 0.240484568927395 -> 0.240484568977745
- link top_stud_link: mass 0.00137057236420411 -> 0.00137057236420412
Joints:
- removed joint robot_body_joint
- removed joint ultrasonic_joint
- added joint camera_optical_joint: type fixed, parent camera_link, child camera_optical_link, origin xyz=-0.0285214690324131 0.0532714690323321 -0.0320399999999404 rpy=-1.5707963267949 0 -1.57079632679491
- added joint ir_back_joint: type fixed, parent base_link, child ir_back_link, origin xyz=0.00389 -0.15402 0.01325 rpy=0 1.5707963267949 0
- added joint ir_front_joint: type fixed, parent base_link, child ir_front_link, origin xyz=-0.36061 -0.14597 0.01325 rpy=0 1.5707963267949 3.1415926535898
- added joint ir_front_left_joint: type fixed, parent base_link, child ir_front_left_link, origin xyz=-0.34189 -0.27041 0.01325 rpy=0 1.5707963267949 -2.3561944901923
- added joint ir_front_right_joint: type fixed, parent base_link, child ir_front_right_link, origin xyz=-0.33619 -0.02391 0.01325 rpy=0 1.5707963267949 2.3561944901923
- added joint ir_left_joint: type fixed, parent base_link, child ir_left_link, origin xyz=-0.16403 -0.30425 0.01325 rpy=0 1.5707963267949 -1.5707963267949
- added joint ir_right_joint: type fixed, parent base_link, child ir_right_link, origin xyz=-0.15593 0.00425 0.01325 rpy=0 1.5707963267949 1.5707963267949
- joint back_right_wheel_joint: axis 0 0 1 -> 0 0 -1
- joint bottom_stud_joint: limit lower=0 upper=0 effort=0 velocity=0 -> lower=-0.05 upper=0.05 effort=150 velocity=0.15
- joint camera_joint: axis 0 0 -1 -> 0 0 1; limit lower=0 upper=0 effort=0 velocity=0 -> lower=-1.5707963268 upper=1.5707963268 effort=10 velocity=2.0; origin xyz=0.117803138552453 0.0228565208887948 0.0849999999999819 rpy=0 0 0 -> xyz=0.11780313855266 0.0228565208888024 0.0850000000000067 rpy=0 0 0
- joint front_right_wheel_joint: axis 0 0 1 -> 0 0 -1
- joint imu_joint: origin xyz=0 0 0.05 rpy=0 0 0 -> xyz=-0.15866 -0.15079 0.010 rpy=0 0 0; parent RobotBody -> base_link
- joint left_joint1: limit lower=0 upper=0 effort=0 velocity=0 -> lower=-0.7853981634 upper=0.7853981634 effort=80 velocity=3.0; origin xyz=0 0.0421507194078778 0 rpy=1.5707963267949 -1.5707963267949 0 -> xyz=0 0.0421507194079047 0 rpy=1.5707963267949 -1.5707963267949 0
- joint left_joint2: limit lower=0 upper=0 effort=0 velocity=0 -> lower=-0.7853981634 upper=0.7853981634 effort=80 velocity=3.0; origin xyz=0.0200000000000404 -0.0374999999999837 0.0424999999994037 rpy=1.5707963267949 0 0 -> xyz=0.0199999999999877 -0.037500000000009 0.0424999999999793 rpy=1.5707963267949 0 0
- joint left_joint3: limit lower=0 upper=0 effort=0 velocity=0 -> lower=-1.5707963268 upper=1.5707963268 effort=80 velocity=3.0; origin xyz=0.117803138552808 0.0228565208880964 0.00499999999999923 rpy=3.14159265358979 0 3.14159265358979 -> xyz=0.117803138552934 0.0228565208874119 0.00500000000000156 rpy=3.14159265358979 0 3.14159265358979
- joint left_joint4: limit lower=0 upper=0 effort=0 velocity=0 -> lower=-1.5707963268 upper=1.5707963268 effort=80 velocity=3.0; origin xyz=0.117803138552813 0.0228565208880835 0.00499999999999956 rpy=3.14159265358979 0 3.14159265358979 -> xyz=0.117803138552674 0.0228565208888156 0.00500000000000111 rpy=3.14159265358979 0 3.14159265358979
- joint left_joint5: limit lower=0 upper=0 effort=0 velocity=0 -> lower=-1.5707963268 upper=1.5707963268 effort=80 velocity=3.0; origin xyz=0.117803138552813 0.0228565208880058 0.00499999999999967 rpy=3.14159265358979 0 3.14159265358979 -> xyz=0.11780313855294 0.0228565208874148 0.00499999999999923 rpy=3.14159265358979 0 3.14159265358979
- joint left_joint6: limit lower=0 upper=0 effort=0 velocity=0 -> lower=-1.5707963268 upper=1.5707963268 effort=80 velocity=3.0; origin xyz=0.11780313855282 0.0228565208881415 0.00499999999999901 rpy=-3.14159265358979 0 -3.14159265358979 -> xyz=0.117803138552671 0.0228565208888066 0.00500000000000234 rpy=-3.14159265358979 0 -3.14159265358979
- joint right_joint1: limit lower=0 upper=0 effort=0 velocity=0 -> lower=-0.7853981634 upper=0.7853981634 effort=80 velocity=3.0; origin xyz=0 -0.0428492805921222 0 rpy=1.5707963267949 -1.5707963267949 0 -> xyz=0 -0.0428492805920998 0 rpy=1.5707963267949 -1.5707963267949 0
- joint right_joint2: limit (none) -> lower=-0.7853981634 upper=0.7853981634 effort=80 velocity=3.0; origin xyz=0.0200000000000368 0.0375000000000166 0.0424999999993435 rpy=1.5707963267949 0 0 -> xyz=0.0199999999999953 0.037499999999994 0.0424999999999847 rpy=1.5707963267949 0 0; type continuous -> revolute
- joint right_joint3: limit lower=0 upper=0 effort=0 velocity=0 -> lower=-1.5707963268 upper=1.5707963268 effort=80 velocity=3.0; origin xyz=0.117803138552811 0.0228565208881228 -0.00500000000000023 rpy=3.14159265358979 0 3.14159265358979 -> xyz=0.117803138552934 0.0228565208874355 -0.00500000000000012 rpy=3.14159265358979 0 3.14159265358979
- joint right_joint4: limit lower=0 upper=0 effort=0 velocity=0 -> lower=-1.5707963268 upper=1.5707963268 effort=80 velocity=3.0; origin xyz=0.117803138552813 0.0228565208880633 -0.00499999999999967 rpy=3.14159265358979 0 3.14159265358979 -> xyz=0.117803138552677 0.022856520888779 -0.00500000000000089 rpy=3.14159265358979 0 3.14159265358979
- joint right_joint5: axis 0 0.259675848455465 -0.965695839138253 -> 0 0 -1; limit lower=0 upper=0 effort=0 velocity=0 -> lower=-1.5707963268 upper=1.5707963268 effort=80 velocity=3.0; origin xyz=0.117803138552815 0.022856520887972 -0.00500000000000012 rpy=2.87890613213286 0 3.14159265358978 -> xyz=0.117803138552938 0.0228565208873703 -0.00499999999999845 rpy=3.14159265358979 0 3.14159265358979
- joint right_joint6: limit lower=0 upper=0 effort=0 velocity=0 -> lower=-1.5707963268 upper=1.5707963268 effort=80 velocity=3.0; origin xyz=0.117803138552816 0.0228565208881623 -0.00499999999999978 rpy=-3.14159265358979 0 -3.14159265358979 -> xyz=0.11780313855268 0.0228565208887971 -0.00500000000000211 rpy=-3.14159265358979 0 -3.14159265358979
- joint top_stud_joint: limit lower=0 upper=0 effort=0 velocity=0 -> lower=-0.05 upper=0.05 effort=150 velocity=0.15; origin xyz=0.117801346067773 0.0228566574753921 -0.0371507194078791 rpy=-1.5707963267949 0 1.5707963267949 -> xyz=0.117801346067551 0.022856657474836 -0.0371507194079034 rpy=-1.5707963267949 0 1.5707963267949

Commit message: full file structure with initial content following the labs

File: src/audix_pkg/urdf/audix.urdf (robot description, URDF)
Before this commit: robot audix, 29 links, 28 joints
Links:
- added link RobotBody
- link back_left_wheel_link: mass 0.131907512521704 -> 0.131907
- link back_right_wheel_link: mass 0.131907120892093 -> 0.131907
- link bottom_stud_link: mass 0.00137057236420413 -> 0.00137057
- link camera_link: mass 0.354470228585855 -> 0.354470
- link front_left_wheel_link: mass 0.131907088712342 -> 0.131907
- link front_right_wheel_link: mass 0.131907397861947 -> 0.131907
- link left_link1: mass 0.00615413438956669 -> 0.006154
- link left_link2: mass 0.00615413438956668 -> 0.006154
- link left_link3: mass 0.00615413438956673 -> 0.006154
- link left_link4: mass 0.00615413438956676 -> 0.006154
- link left_link5: mass 0.00615413438956676 -> 0.006154
- link left_link6: mass 0.00615413438956674 -> 0.006154
- link right_link1: mass 0.00615413438956677 -> 0.006154
- link right_link2: mass 0.00615413438956663 -> 0.006154
- link right_link3: mass 0.00615413438956681 -> 0.006154
- link right_link4: mass 0.00615413438956673 -> 0.006154
- link right_link5: mass 0.00615413438956677 -> 0.006154
- link right_link6: mass 0.0061541343895667 -> 0.006154
- link top_stud_link: mass 0.00137057236420412 -> 0.001371
Joints:
- added joint robot_body_joint: type fixed, parent base_link, child RobotBody, origin xyz=0 0 0 rpy=0 0 0
- joint bottom_stud_joint: limit lower=-0.05 upper=0.05 effort=150 velocity=0.15 -> lower=0.0 upper=0.0772 effort=150 velocity=0.05
- joint camera_joint: limit lower=-1.5707963268 upper=1.5707963268 effort=10 velocity=2.0 -> lower=-1.5708 upper=1.5708 effort=10 velocity=2.0
- joint left_joint1: limit lower=-0.7853981634 upper=0.7853981634 effort=80 velocity=3.0 -> lower=-1.5708 upper=1.5708 effort=80 velocity=3.0
- joint left_joint2: limit lower=-0.7853981634 upper=0.7853981634 effort=80 velocity=3.0 -> lower=-1.5708 upper=1.5708 effort=80 velocity=3.0
- joint left_joint3: limit lower=-1.5707963268 upper=1.5707963268 effort=80 velocity=3.0 -> lower=-1.5708 upper=1.5708 effort=80 velocity=3.0
- joint left_joint4: limit lower=-1.5707963268 upper=1.5707963268 effort=80 velocity=3.0 -> lower=-1.5708 upper=1.5708 effort=80 velocity=3.0
- joint left_joint5: limit lower=-1.5707963268 upper=1.5707963268 effort=80 velocity=3.0 -> lower=-1.5708 upper=1.5708 effort=80 velocity=3.0
- joint left_joint6: limit lower=-1.5707963268 upper=1.5707963268 effort=80 velocity=3.0 -> lower=-1.5708 upper=1.5708 effort=80 velocity=3.0
- joint right_joint1: limit lower=-0.7853981634 upper=0.7853981634 effort=80 velocity=3.0 -> lower=-1.5708 upper=1.5708 effort=80 velocity=3.0
- joint right_joint2: limit lower=-0.7853981634 upper=0.7853981634 effort=80 velocity=3.0 -> lower=-1.5708 upper=1.5708 effort=80 velocity=3.0
- joint right_joint3: limit lower=-1.5707963268 upper=1.5707963268 effort=80 velocity=3.0 -> lower=-1.5708 upper=1.5708 effort=80 velocity=3.0
- joint right_joint4: limit lower=-1.5707963268 upper=1.5707963268 effort=80 velocity=3.0 -> lower=-1.5708 upper=1.5708 effort=80 velocity=3.0
- joint right_joint5: limit lower=-1.5707963268 upper=1.5707963268 effort=80 velocity=3.0 -> lower=-1.5708 upper=1.5708 effort=80 velocity=3.0
- joint right_joint6: limit lower=-1.5707963268 upper=1.5707963268 effort=80 velocity=3.0 -> lower=-1.5708 upper=1.5708 effort=80 velocity=3.0
- joint scissors_lift_base_fix: axis 0 0 0 -> (none)

Commit message: Update Gazebo launch, scissor mapping, and URDF alignment fixes

File: src/audix_pkg/urdf/audix.urdf (robot description, URDF)
Before this commit: robot audix, 29 links, 28 joints
Links:
- added link base_footprint
Joints:
- added joint base_footprint_joint: type fixed, parent base_footprint, child base_link, origin xyz=0 0 0 rpy=0 0 0
- joint right_joint5: origin xyz=0.117803138552938 0.0228565208873703 -0.00499999999999845 rpy=3.14159265358979 0 3.14159265358979 -> xyz=0.11780313855294 0.0228565208874148 -0.00499999999999923 rpy=3.14159265358979 0 3.14159265358979

Commit message: bta3i

File: src/audix_pkg/urdf/audix.urdf (robot description, URDF)
Before this commit: robot audix, 30 links, 29 joints
Links:
- link back_left_wheel_link: geometry collision cylinder length=0.025 radius=0.0485; visual mesh filename=package://audix/meshes/back_left_wheel_link.STL
- link back_right_wheel_link: geometry collision cylinder length=0.025 radius=0.0485; visual mesh filename=package://audix/meshes/back_right_wheel_link.STL
- link base_link: geometry collision box size=0.32 0.35 0.11; visual mesh filename=package://audix/meshes/base_link.STL
- link bottom_stud_link: geometry collision cylinder length=0.015 radius=0.004; visual mesh filename=package://audix/meshes/bottom_stud_link.STL
- link camera_link: geometry collision box size=0.15 0.12 0.10; visual mesh filename=package://audix/meshes/camera_link.STL
- link front_left_wheel_link: geometry collision cylinder length=0.025 radius=0.0485; visual mesh filename=package://audix/meshes/front_left_wheel_link.STL
- link front_right_wheel_link: geometry collision cylinder length=0.025 radius=0.0485; visual mesh filename=package://audix/meshes/front_right_wheel_link.STL
- link left_link1: geometry collision box size=0.12 0.015 0.012; visual mesh filename=package://audix/meshes/left_link1.STL
- link left_link2: geometry collision box size=0.12 0.015 0.012; visual mesh filename=package://audix/meshes/left_link2.STL
- link left_link3: geometry collision box size=0.12 0.015 0.012; visual mesh filename=package://audix/meshes/left_link3.STL
- link left_link4: geometry collision box size=0.12 0.015 0.012; visual mesh filename=package://audix/meshes/left_link4.STL
- link left_link5: geometry collision box size=0.12 0.015 0.012; visual mesh filename=package://audix/meshes/left_link5.STL
- link left_link6: geometry collision box size=0.12 0.015 0.012; visual mesh filename=package://audix/meshes/left_link6.STL
- link right_link1: geometry collision box size=0.12 0.015 0.012; visual mesh filename=package://audix/meshes/right_link1.STL
- link right_link2: geometry collision box size=0.12 0.015 0.012; visual mesh filename=package://audix/meshes/right_link2.STL
- link right_link3: geometry collision box size=0.12 0.015 0.012; visual mesh filename=package://audix/meshes/right_link3.STL
- link right_link4: geometry collision box size=0.12 0.015 0.012; visual mesh filename=package://audix/meshes/right_link4.STL
- link right_link5: geometry collision box size=0.12 0.015 0.012; visual mesh filename=package://audix/meshes/right_link5.STL
- link right_link6: geometry collision box size=0.12 0.015 0.012; visual mesh filename=package://audix/meshes/right_link6.STL
- link scissors_lift_base: geometry collision box size=0.22 0.10 0.08; visual mesh filename=package://audix/meshes/scissors_lift_base.STL
- link top_stud_link: geometry collision cylinder length=0.015 radius=0.004; visual mesh filename=package://audix/meshes/top_stud_link.STL

Commit message: Robot moves but the waypoints are still not clear

File: src/audix_pkg/urdf/audix.urdf (robot description, URDF)
Before this commit: robot audix, 30 links, 29 joints
Joints:
- joint robot_body_joint: origin xyz=0 0 0 rpy=0 0 0 -> xyz=0 0 0 rpy=0 0 3.14159

Commit message: missing only obstacle avoidance

File: src/audix_pkg/urdf/audix.urdf (robot description, URDF)
Before this commit: robot audix, 30 links, 29 joints
Links:
- removed link RobotBody
- added link base_footprint
- link back_left_wheel_link: mass 0.131907 -> 0.131907512521704; geometry collision mesh filename=package://audix/meshes/back_left_wheel_link.STL; visual mesh filename=package://audix/meshes/back_left_wheel_link.STL
- link back_right_wheel_link: mass 0.131907 -> 0.131907120892093; geometry collision mesh filename=package://audix/meshes/back_right_wheel_link.STL; visual mesh filename=package://audix/meshes/back_right_wheel_link.STL
- link base_link: geometry collision mesh filename=package://audix/meshes/base_link.STL; visual mesh filename=package://audix/meshes/base_link.STL
- link bottom_stud_link: mass 0.00137057 -> 0.00137057236420413; geometry collision mesh filename=package://audix/meshes/bottom_stud_link.STL; visual mesh filename=package://audix/meshes/bottom_stud_link.STL
- link camera_link: mass 0.354470 -> 0.354470228585855; geometry collision mesh filename=package://audix/meshes/camera_link.STL; visual mesh filename=package://audix/meshes/camera_link.STL
- link front_left_wheel_link: mass 0.131907 -> 0.131907088712342; geometry collision mesh filename=package://audix/meshes/front_left_wheel_link.STL; visual mesh filename=package://audix/meshes/front_left_wheel_link.STL
- link front_right_wheel_link: mass 0.131907 -> 0.131907397861947; geometry collision mesh filename=package://audix/meshes/front_right_wheel_link.STL; visual mesh filename=package://audix/meshes/front_right_wheel_link.STL
- link left_link1: mass 0.006154 -> 0.00615413438956669; geometry collision mesh filename=package://audix/meshes/left_link1.STL; visual mesh filename=package://audix/meshes/left_link1.STL
- link left_link2: mass 0.006154 -> 0.00615413438956668; geometry collision mesh filename=package://audix/meshes/left_link2.STL; visual mesh filename=package://audix/meshes/left_link2.STL
- link left_link3: mass 0.006154 -> 0.00615413438956673; geometry collision mesh filename=package://audix/meshes/left_link3.STL; visual mesh filename=package://audix/meshes/left_link3.STL
- link left_link4: mass 0.006154 -> 0.00615413438956676; geometry collision mesh filename=package://audix/meshes/left_link4.STL; visual mesh filename=package://audix/meshes/left_link4.STL
- link left_link5: mass 0.006154 -> 0.00615413438956676; geometry collision mesh filename=package://audix/meshes/left_link5.STL; visual mesh filename=package://audix/meshes/left_link5.STL
- link left_link6: mass 0.006154 -> 0.00615413438956674; geometry collision mesh filename=package://audix/meshes/left_link6.STL; visual mesh filename=package://audix/meshes/left_link6.STL
- link right_link1: mass 0.006154 -> 0.00615413438956677; geometry collision mesh filename=package://audix/meshes/right_link1.STL; visual mesh filename=package://audix/meshes/right_link1.STL
- link right_link2: mass 0.006154 -> 0.00615413438956663; geometry collision mesh filename=package://audix/meshes/right_link2.STL; visual mesh filename=package://audix/meshes/right_link2.STL
- link right_link3: mass 0.006154 -> 0.00615413438956681; geometry collision mesh filename=package://audix/meshes/right_link3.STL; visual mesh filename=package://audix/meshes/right_link3.STL
- link right_link4: mass 0.006154 -> 0.00615413438956673; geometry collision mesh filename=package://audix/meshes/right_link4.STL; visual mesh filename=package://audix/meshes/right_link4.STL
- link right_link5: mass 0.006154 -> 0.00615413438956677; geometry collision mesh filename=package://audix/meshes/right_link5.STL; visual mesh filename=package://audix/meshes/right_link5.STL
- link right_link6: mass 0.006154 -> 0.0061541343895667; geometry collision mesh filename=package://audix/meshes/right_link6.STL; visual mesh filename=package://audix/meshes/right_link6.STL
- link scissors_lift_base: geometry collision mesh filename=package://audix/meshes/scissors_lift_base.STL; visual mesh filename=package://audix/meshes/scissors_lift_base.STL
- link top_stud_link: mass 0.001371 -> 0.00137057236420412; geometry collision mesh filename=package://audix/meshes/top_stud_link.STL; visual mesh filename=package://audix/meshes/top_stud_link.STL
Joints:
- removed joint robot_body_joint
- added joint base_footprint_joint: type fixed, parent base_footprint, child base_link, origin xyz=0 0 0 rpy=0 0 0
- joint bottom_stud_joint: limit lower=0.0 upper=0.0772 effort=150 velocity=0.05 -> lower=-0.05 upper=0.05 effort=150 velocity=0.15
- joint camera_joint: limit lower=-1.5708 upper=1.5708 effort=10 velocity=2.0 -> lower=-1.5707963268 upper=1.5707963268 effort=10 velocity=2.0
- joint left_joint1: limit lower=-1.5708 upper=1.5708 effort=80 velocity=3.0 -> lower=-0.7853981634 upper=0.7853981634 effort=80 velocity=3.0
- joint left_joint2: limit lower=-1.5708 upper=1.5708 effort=80 velocity=3.0 -> lower=-0.7853981634 upper=0.7853981634 effort=80 velocity=3.0
- joint left_joint3: limit lower=-1.5708 upper=1.5708 effort=80 velocity=3.0 -> lower=-1.5707963268 upper=1.5707963268 effort=80 velocity=3.0
- joint left_joint4: limit lower=-1.5708 upper=1.5708 effort=80 velocity=3.0 -> lower=-1.5707963268 upper=1.5707963268 effort=80 velocity=3.0
- joint left_joint5: limit lower=-1.5708 upper=1.5708 effort=80 velocity=3.0 -> lower=-1.5707963268 upper=1.5707963268 effort=80 velocity=3.0
- joint left_joint6: limit lower=-1.5708 upper=1.5708 effort=80 velocity=3.0 -> lower=-1.5707963268 upper=1.5707963268 effort=80 velocity=3.0
- joint right_joint1: limit lower=-1.5708 upper=1.5708 effort=80 velocity=3.0 -> lower=-0.7853981634 upper=0.7853981634 effort=80 velocity=3.0
- joint right_joint2: limit lower=-1.5708 upper=1.5708 effort=80 velocity=3.0 -> lower=-0.7853981634 upper=0.7853981634 effort=80 velocity=3.0
- joint right_joint3: limit lower=-1.5708 upper=1.5708 effort=80 velocity=3.0 -> lower=-1.5707963268 upper=1.5707963268 effort=80 velocity=3.0
- joint right_joint4: limit lower=-1.5708 upper=1.5708 effort=80 velocity=3.0 -> lower=-1.5707963268 upper=1.5707963268 effort=80 velocity=3.0
- joint right_joint5: limit lower=-1.5708 upper=1.5708 effort=80 velocity=3.0 -> lower=-1.5707963268 upper=1.5707963268 effort=80 velocity=3.0; origin xyz=0.117803138552938 0.0228565208873703 -0.00499999999999845 rpy=3.14159265358979 0 3.14159265358979 -> xyz=0.11780313855294 0.0228565208874148 -0.00499999999999923 rpy=3.14159265358979 0 3.14159265358979
- joint right_joint6: limit lower=-1.5708 upper=1.5708 effort=80 velocity=3.0 -> lower=-1.5707963268 upper=1.5707963268 effort=80 velocity=3.0
- joint scissors_lift_base_fix: axis (none) -> 0 0 0
